Commit message: Worked on state stuff

File: ros/src/msurobosub/robosub_model.urdf (robot description, URDF)
Before this commit: robot robosub, 4 links, 3 joints
Links:
- added link cameraD; visual box size=.05 .05 .05
- added link cameraF; visual box size=.05 .05 .05
- added link imu0; visual box size=.05 .05 .05
Joints:
- added joint base_to_camD: type fixed, parent base_link, child cameraD, origin xyz=0 0 -.3 rpy=0 0 0
- added joint base_to_camF: type fixed, parent base_link, child cameraF, origin xyz=0 .5 0 rpy=0 0 0
- added joint base_to_imu0: type fixed, parent base_link, child imu0, origin xyz=.1 -.3 0 rpy=0 0 0
- joint base_to_torp1: origin xyz=-0.1 0.3 0.2 rpy=0 0 0 -> xyz=-0.1 0.3 0.2 rpy=1.5708 0 0
- joint base_to_torp2: origin xyz=0.1 0.3 0.2 rpy=0 0 0 -> xyz=0.1 0.3 0.2 rpy=1.5708 0 0
